File: duncan_kelley/duncan_kelley.kicad_sch (KiCad schematic)
At the start: 14 parts, among them J1 RJ45_LED_Shielded, SW1 SW_Push, U1 OKI, U2 Teensy4.1_DEV-16771

Commit message: uh yeah it's done
Parts:
- C1, C2, C3: footprint (none) -> Capacitor_SMD:C_0603_1608Metric_Pad1.08x0.95mm_HandSolder
- Conn1: footprint (none) -> MRDT_Connectors:Square_Anderson_2_H_Side_By_Side_PV
- D1, D2, D3: footprint (none) -> Diode_SMD:D_0603_1608Metric_Pad1.05x0.95mm_HandSolder
- J1: footprint (none) -> MRDT_Connectors:RJ45_Teensy
- R1, R2, R3: footprint (none) -> Resistor_SMD:R_0603_1608Metric_Pad0.98x0.95mm_HandSolder
- SW1: footprint (none) -> Button_Switch_SMD:SW_SPST_TL3305A
- U1: footprint (none) -> MRDT_Devices:OKI_Horizontal
- U2: footprint MODULE_DEV-16771 -> MRDT_Shields:Teensy_4_1
Changed lines of the file:
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@@
     (pin "1")
     (instances
-      (project "duncankelley"
+      (project "duncan_kelley"
         (path "/db90db77-1fcf-47bb-acb2-4fc76581a666"
           (reference "#PWR09") (unit 1)
@@
       (effects (font (size 1.27 1.27)))
     )
-    (property "Footprint" "" (at 115.57 84.328 90)
+    (property "Footprint" "Resistor_SMD:R_0603_1608Metric_Pad0.98x0.95mm_HandSolder" (at 115.57 84.328 90)
       (effects (font (size 1.27 1.27)) hide)
     )
@@
     (pin "2")
     (instances
-      (project "duncankelley"
+      (project "duncan_kelley"
         (path "/db90db77-1fcf-47bb-acb2-4fc76581a666"
           (reference "R3") (unit 1)
@@
     (pin "1")
     (instances
-      (project "duncankelley"
+      (project "duncan_kelley"
         (path "/db90db77-1fcf-47bb-acb2-4fc76581a666"
           (reference "#PWR02") (unit 1)
@@
       (effects (font (size 1.27 1.27)))
     )
-    (property "Footprint" "" (at 127 82.55 0)
+    (property "Footprint" "Diode_SMD:D_0603_1608Metric_Pad1.05x0.95mm_HandSolder" (at 127 82.55 0)
       (effects (font (size 1.27 1.27)) hide)
     )
@@
     (pin "2")
     (instances
-      (project "duncankelley"
+      (project "duncan_kelley"
         (path "/db90db77-1fcf-47bb-acb2-4fc76581a666"
           (reference "D3") (unit 1)
@@
       (effects (font (size 1.27 1.27)) (justify left))
     )
-    (property "Footprint" "" (at 49.2252 81.28 0)
+    (property "Footprint" "Capacitor_SMD:C_0603_1608Metric_Pad1.08x0.95mm_HandSolder" (at 49.2252 81.28 0)
       (effects (font (size 1.27 1.27)) hide)
     )
@@
     (pin "2")
     (instances
-      (project "duncankelley"
+      (project "duncan_kelley"
         (path "/db90db77-1fcf-47bb-acb2-4fc76581a666"
           (reference "C1") (unit 1)
@@
     (pin "1")
     (instances
-      (project "duncankelley"
+      (project "duncan_kelley"
         (path "/db90db77-1fcf-47bb-acb2-4fc76581a666"
           (reference "#PWR08") (unit 1)
@@
     (pin "1")
     (instances
-      (project "duncankelley"
+      (project "duncan_kelley"
         (path "/db90db77-1fcf-47bb-acb2-4fc76581a666"
           (reference "#PWR011") (unit 1)
@@
       (effects (font (size 1.27 1.27)) (justify right))
     )
-    (property "Footprint" "" (at 123.19 43.18 0)
+    (property "Footprint" "Diode_SMD:D_0603_1608Metric_Pad1.05x0.95mm_HandSolder" (at 123.19 43.18 0)
       (effects (font (size 1.27 1.27)) hide)
     )
@@
     (pin "2")
     (instances
-      (project "duncankelley"
+      (project "duncan_kelley"
         (path "/db90db77-1fcf-47bb-acb2-4fc76581a666"
           (reference "D2") (unit 1)
@@
     (pin "1")
     (instances
-      (project "duncankelley"
+      (project "duncan_kelley"
         (path "/db90db77-1fcf-47bb-acb2-4fc76581a666"
           (reference "#PWR01") (unit 1)
@@
       (effects (font (size 1.27 1.27)))
     )
-    (property "Footprint" "" (at 259.08 51.435 90)
+    (property "Footprint" "MRDT_Connectors:RJ45_Teensy" (at 259.08 51.435 90)
       (effects (font (size 1.27 1.27)) hide)
     )
@@
     (pin "SH")
     (instances
-      (project "duncankelley"
+      (project "duncan_kelley"
         (path "/db90db77-1fcf-47bb-acb2-4fc76581a666"
           (reference "J1") (unit 1)
@@
       (effects (font (size 1.27 1.27)))
     )
-    (property "Footprint" "" (at 102.87 77.47 0)
+    (property "Footprint" "Button_Switch_SMD:SW_SPST_TL3305A" (at 102.87 77.47 0)
       (effects (font (size 1.27 1.27)) hide)
     )
@@
     (pin "2")
     (instances
-      (project "duncankelley"
+      (project "duncan_kelley"
         (path "/db90db77-1fcf-47bb-acb2-4fc76581a666"
           (reference "SW1") (unit 1)
@@
       (effects (font (size 1.27 1.27)))
     )
-    (property "Footprint" "" (at 241.3 52.3748 0)
+    (property "Footprint" "Capacitor_SMD:C_0603_1608Metric_Pad1.08x0.95mm_HandSolder" (at 241.3 52.3748 0)
       (effects (font (size 1.27 1.27)) hide)
     )
@@
     (pin "2")
     (instances
-      (project "duncankelley"
+      (project "duncan_kelley"
         (path "/db90db77-1fcf-47bb-acb2-4fc76581a666"
           (reference "C3") (unit 1)
@@
     (pin "1")
     (instances
-      (project "duncankelley"
+      (project "duncan_kelley"
         (path "/db90db77-1fcf-47bb-acb2-4fc76581a666"
           (reference "#PWR07") (unit 1)
@@
     (pin "1")
     (instances
-      (project "duncankelley"
+      (project "duncan_kelley"
         (path "/db90db77-1fcf-47bb-acb2-4fc76581a666"
           (reference "#PWR010") (unit 1)
@@
       (effects (font (size 1.524 1.524)))
     )
-    (property "Footprint" "" (at 25.4 77.47 0)
+    (property "Footprint" "MRDT_Devices:OKI_Horizontal" (at 25.4 77.47 0)
       (effects (font (size 1.524 1.524)) hide)
     )
@@
     (pin "3")
     (instances
-      (project "duncankelley"
+      (project "duncan_kelley"
         (path "/db90db77-1fcf-47bb-acb2-4fc76581a666"
           (reference "U1") (unit 1)
@@
     (pin "1")
     (instances
-      (project "duncankelley"
+      (project "duncan_kelley"
         (path "/db90db77-1fcf-47bb-acb2-4fc76581a666"
           (reference "#PWR03") (unit 1)
@@
       (effects (font (size 1.524 1.524)))
     )
-    (property "Footprint" "" (at 27.94 48.26 0)
+    (property "Footprint" "MRDT_Connectors:Square_Anderson_2_H_Side_By_Side_PV" (at 27.94 48.26 0)
       (effects (font (size 1.524 1.524)) hide)
     )
@@
     (pin "1")
     (instances
-      (project "duncankelley"
+      (project "duncan_kelley"
         (path "/db90db77-1fcf-47bb-acb2-4fc76581a666"
           (reference "Conn1") (unit 4)
@@
       (effects (font (size 1.27 1.27)))
     )
-    (property "Footprint" "MODULE_DEV-16771" (at 260.35 88.9 0)
+    (property "Footprint" "MRDT_Shields:Teensy_4_1" (at 260.35 88.9 0)
       (effects (font (size 1.27 1.27)) (justify left bottom) hide)
     )
@@
     (pin "VUSB")
     (instances
-      (project "duncankelley"
+      (project "duncan_kelley"
         (path "/db90db77-1fcf-47bb-acb2-4fc76581a666"
           (reference "U2") (unit 1)
@@
     (pin "1")
     (instances
-      (project "duncankelley"
+      (project "duncan_kelley"
         (path "/db90db77-1fcf-47bb-acb2-4fc76581a666"
           (reference "#PWR04") (unit 1)
@@
       (effects (font (size 1.27 1.27)) (justify left))
     )
-    (property "Footprint" "" (at 106.172 33.02 90)
+    (property "Footprint" "Resistor_SMD:R_0603_1608Metric_Pad0.98x0.95mm_HandSolder" (at 106.172 33.02 90)
       (effects (font (size 1.27 1.27)) hide)
     )
@@
     (pin "2")
     (instances
-      (project "duncankelley"
+      (project "duncan_kelley"
         (path "/db90db77-1fcf-47bb-acb2-4fc76581a666"
           (reference "R1") (unit 1)
@@
       (effects (font (size 1.27 1.27)) (justify left))
     )
-    (property "Footprint" "" (at 23.8252 81.28 0)
+    (property "Footprint" "Capacitor_SMD:C_0603_1608Metric_Pad1.08x0.95mm_HandSolder" (at 23.8252 81.28 0)
       (effects (font (size 1.27 1.27)) hide)
     )
@@
     (pin "2")
     (instances
-      (project "duncankelley"
+      (project "duncan_kelley"
         (path "/db90db77-1fcf-47bb-acb2-4fc76581a666"
           (reference "C2") (unit 1)
@@
       (effects (font (size 1.524 1.524)))
     )
-    (property "Footprint" "" (at 27.94 60.96 0)
+    (property "Footprint" "MRDT_Connectors:Square_Anderson_2_H_Side_By_Side_PV" (at 27.94 60.96 0)
       (effects (font (size 1.524 1.524)) hide)
     )
@@
     (pin "1")
     (instances
-      (project "duncankelley"
+      (project "duncan_kelley"
         (path "/db90db77-1fcf-47bb-acb2-4fc76581a666"
           (reference "Conn1") (unit 1)
@@
     (pin "1")
     (instances
-      (project "duncankelley"
+      (project "duncan_kelley"
         (path "/db90db77-1fcf-47bb-acb2-4fc76581a666"
           (reference "#PWR06") (unit 1)
@@
       (effects (font (size 1.27 1.27)) (justify right))
     )
-    (property "Footprint" "" (at 107.95 43.18 0)
+    (property "Footprint" "Diode_SMD:D_0603_1608Metric_Pad1.05x0.95mm_HandSolder" (at 107.95 43.18 0)
       (effects (font (size 1.27 1.27)) hide)
     )
@@
     (pin "2")
     (instances
-      (project "duncankelley"
+      (project "duncan_kelley"
         (path "/db90db77-1fcf-47bb-acb2-4fc76581a666"
           (reference "D1") (unit 1)
@@
     (pin "1")
     (instances
-      (project "duncankelley"
+      (project "duncan_kelley"
         (path "/db90db77-1fcf-47bb-acb2-4fc76581a666"
           (reference "#PWR05") (unit 1)
@@
       (effects (font (size 1.27 1.27)) (justify left))
     )
-    (property "Footprint" "" (at 121.412 33.02 90)
+    (property "Footprint" "Resistor_SMD:R_0603_1608Metric_Pad0.98x0.95mm_HandSolder" (at 121.412 33.02 90)
       (effects (font (size 1.27 1.27)) hide)
     )
@@
     (pin "2")
     (instances
-      (project "duncankelley"
+      (project "duncan_kelley"
         (path "/db90db77-1fcf-47bb-acb2-4fc76581a666"
           (reference "R2") (unit 1)
