File: Hardware/Dylan Dush/DylanDush - Training Hardware/_autosave-DylanDush - Training Hardware.kicad_sch (KiCad schematic)
At the start: 14 parts, among them J1 RJ45_LED_Shielded, SW1 SW_Push, U1 OKI, U2 Teensy4.1_DEV-16771

Commit message: Layout Training complete
Learned dat junks
Connections:
- net R+: now reaches J1.4, U2.R+
- net R-: now reaches J1.6, U2.R-
- net T+: now reaches J1.1, U2.T+
- net T-: now reaches J1.3, U2.T-
Changed lines of the file:
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@@
     (effects (font (size 2.54 2.54)) (justify left bottom))
+  )
+  (label "R-" (at 135.255 46.99 0) (fields_autoplaced)
+    (effects (font (size 1.27 1.27)) (justify left bottom))
+  )
+  (label "T+" (at 135.255 44.45 0) (fields_autoplaced)
+    (effects (font (size 1.27 1.27)) (justify left bottom))
+  )
+  (label "R+" (at 135.255 49.53 0) (fields_autoplaced)
+    (effects (font (size 1.27 1.27)) (justify left bottom))
+  )
+  (label "T-" (at 135.255 41.91 0) (fields_autoplaced)
+    (effects (font (size 1.27 1.27)) (justify left bottom))
   )
   (global_label "PV" (shape output) (at 54.61 31.75 0) (fields_autoplaced)
