File: Hardware/niko_hidayat/Niko Hidayat.kicad_sch (KiCad schematic)
At the start: 14 parts, among them J1 8P8C_LED_Shielded, SW1 SW_Push, U1 OKI, U2 Teensy4.1_DEV-16771

Commit message: Layout Training Complete
:)
Connections:
- net R+: now reaches J1.4, U2.R+
- net R-: now reaches J1.6, U2.R-
Changed lines of the file:
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@@
     (effects (font (size 5.08 5.08)) (justify left bottom))
+  )
+  (label "R-" (at 215.9 53.34 0) (fields_autoplaced)
+    (effects (font (size 1.27 1.27)) (justify left bottom))
+  )
+  (label "R+" (at 215.9 55.88 0) (fields_autoplaced)
+    (effects (font (size 1.27 1.27)) (justify left bottom))
   )
   (label "T-" (at 215.9 48.26 0) (fields_autoplaced)
